File: Board/shoe_5/shoe_5.kicad_pcb (KiCad board)
At the start: 2 copper layers, 33 parts, among them SW1 SW_DIP_x01, U1 LMV324, U2 LMV324, U3 WeMos_mini

Commit message: checking day 18/07
Parts:
- added C10: 470uF, Capacitor_THT:CP_Radial_D5.0mm_P2.50mm, F.Cu at (43.2, 43.8)
- C6: value CP -> 100uF
- RV1: footprint Potentiometer_THT:Potentiometer_Bourns_3296W_Vertical -> Potentiometer_THT:Potentiometer_Bourns_3006P_Horizontal
- SW1: footprint myfootprint:SW -> myfootprint:SW_small
- moved V1 49.9 mm to (80.5, 42.0)
- moved C6 17.9 mm to (17.0, 103.0)
- moved C4 10.7 mm to (16.7, 89.2)
- moved C5 10.7 mm to (24.2, 89.2)
- moved RV1 9.17 mm to (52.0, 91.8)
- moved SW1 0.35 mm to (22.8, 49.2)
Connections:
- BT1 pad 1: /Source -> Net-(BT1-Pad1)
- SW1 pad 1: /Source -> Net-(BT1-Pad1)
- SW1 pad 2: Net-(SW1-Pad2) -> /Source
- V1 pad 1: Net-(SW1-Pad2) -> /Source
