File: Board/shoe_5/shoe_5.sch (KiCad schematic (older format))
At the start: 41 parts

Commit message: please do more wiring
Parts:
- removed AG?: GY-25, symbol shoe_2:GY-25
- removed U? (x10): LM324, symbol Amplifier_Operational:LM324
- removed U?: ESP-12F, RF_Module:ESP-12E, symbol RF_Module:ESP-12F
- added MPU1: MPU9250, Connector_PinSocket_2.54mm:PinSocket_1x10_P2.54mm_Vertical, symbol shoe_2:MPU9250
- added U1, U2: LMV324, Package_SO:SOIC-14_3.9x8.7mm_P1.27mm, symbol Amplifier_Operational:LMV324
- added U3: WeMos_mini, wemos-d1-mini:wemos-d1-mini-with-pin-header-and-connector, symbol wemos_mini:WeMos_mini
- Adc1, Adc2: renamed from Adc?; footprint (none) -> Connector_PinSocket_2.54mm:PinSocket_1x10_P2.54mm_Vertical
- BT1: renamed from BT?; footprint (none) -> Connector_PinSocket_2.54mm:PinSocket_2x01_P2.54mm_Vertical
- C1, C2, C3, C7, C8, C9: renamed from C?; footprint (none) -> Capacitor_SMD:C_0805_2012Metric
- C4, C5: renamed from C?; footprint (none) -> Capacitor_THT:CP_Radial_Tantal_D4.5mm_P5.00mm
- C6: renamed from C?; footprint (none) -> Capacitor_THT:CP_Radial_D5.0mm_P2.50mm
- R1, R2, R3, R4, R5, R6, R7, R8: renamed from R?; footprint (none) -> Resistor_SMD:R_0805_2012Metric
- RV1: renamed from RV?; footprint (none) -> Potentiometer_THT:Potentiometer_Bourns_3296W_Vertical
- S1, S2, S3, S4, S5, S6: renamed from S?; footprint (none) -> Connector_Wire:SolderWirePad_1x02_P3.81mm_Drill1.2mm
- SW1: renamed from SW?; footprint (none) -> myfootprint:SW
- V1: renamed from V?; footprint (none) -> myfootprint:MT3608_module
Connections:
- net 2v: now also U1.6 (-), U1.7
- net 4v: now also U1.1, U1.10 (+), U1.12 (+), U1.2 (-), U2.10 (+), U2.12 (+), U2.3 (+), U2.5 (+)
- net 8V: now also U1.4 (V+), U2.4 (V+)
- net GND: now also MPU1.2 (GND), U1.11 (V-), U2.11 (V-), U3.2 (GND)
- net SCL: now also MPU1.3 (SCL), U3.6 (D1)
- net SDA: now also MPU1.4 (SDA), U3.5 (D2)
- net Sen_1: now also U1.8
- net Sen_2: now also U2.1
- net Sen_3: now also U2.8
- net Sen_4: now also U1.14
- net Sen_5: now also U2.7
- net Sen_6: now also U2.14
- net Source: now also MPU1.1 (VCC), U3.1 (5V)
- net at R1.2, R2.1: now also U1.3 (+)
- net at RV1.2: now also U1.5 (+)
- net at C1.2, R3.2, S1.1 (Lf): now also U1.9 (-)
- net at C2.2, R4.2, S2.1 (Lf): now also U2.2 (-)
- net at C7.2, R6.2, S4.1 (Lf): now also U1.13 (-)
- net at C8.2, R7.2, S5.1 (Lf): now also U2.6 (-)
- net at C3.2, R5.2, S3.1 (Lf): now also U2.9 (-)
- net at C9.2, R8.2, S6.1 (Lf): now also U2.13 (-)
Other:
- moved on the sheet: C1, C2, C7, C8, R3, R4, R6, R7, S1, S2, S4, S5

Commit message: checking day 18/07
Parts:
- added C10: 470uF, Capacitor_THT:CP_Radial_D5.0mm_P2.50mm, symbol Device:CP
- C6: value CP -> 100uF
- RV1: footprint Potentiometer_THT:Potentiometer_Bourns_3296W_Vertical -> Potentiometer_THT:Potentiometer_Bourns_3006P_Horizontal
- S1, S2, S3, S4, S5, S6: footprint Connector_Wire:SolderWirePad_1x02_P3.81mm_Drill1.2mm -> Connector_PinSocket_2.00mm:PinSocket_1x02_P2.00mm_Horizontal
- SW1: footprint myfootprint:SW -> myfootprint:SW_small
Connections:
- net GND: now also C10.2
- net Source: now also SW1.2, V1.1 (VIN+), C10.1; no longer BT1.1 (+), SW1.1
- new net: BT1.1 (+), SW1.1
Other:
- moved on the sheet: SW1
Changed lines of the file:
@@
 L Switch:SW_DIP_x01 SW1
 U 1 1 5D12705E
-P 1300 800
-F 0 "SW1" H 1300 1067 50  0000 C CNN
-F 1 "SW_DIP_x01" H 1300 976 50  0000 C CNN
-F 2 "myfootprint:SW" H 1300 800 50  0001 C CNN
-F 3 "" H 1300 800 50  0001 C CNN
-	1    1300 800
-	1    0    0    -1
-$EndComp
-Wire Wire Line
-	800  800  1000 800
+P 1100 800
+F 0 "SW1" H 1100 1067 50  0000 C CNN
+F 1 "SW_DIP_x01" H 1100 976 50  0000 C CNN
+F 2 "myfootprint:SW_small" H 1100 800 50  0001 C CNN
+F 3 "" H 1100 800 50  0001 C CNN
+	1    1100 800
+	1    0    0    -1
+$EndComp
 $Comp
 L power:GND #PWR01
@@
 $EndComp
 Wire Wire Line
-	1600 800  1700 800
+	1400 800  1450 800
 Wire Wire Line
 	1700 900  1700 1200
 Wire Wire Line
-	1700 1200 800  1200
+	1700 1200 1450 1200
 Connection ~ 800  1200
 Wire Wire Line
@@
 P 2700 950
 F 0 "C6" H 2818 996 50  0000 L CNN
-F 1 "CP" H 2818 905 50  0000 L CNN
+F 1 "100uF" H 2818 905 50  0000 L CNN
 F 2 "Capacitor_THT:CP_Radial_D5.0mm_P2.50mm" H 2738 800 50  0001 C CNN
 F 3 "" H 2700 950 50  0001 C CNN
@@
 F 0 "RV1" H 2530 2296 50  0000 R CNN
 F 1 "R_POT" H 2530 2205 50  0000 R CNN
-F 2 "Potentiometer_THT:Potentiometer_Bourns_3296W_Vertical" H 2600 2250 50  0001 C CNN
+F 2 "Potentiometer_THT:Potentiometer_Bourns_3006P_Horizontal" H 2600 2250 50  0001 C CNN
 F 3 "" H 2600 2250 50  0001 C CNN
 	1    2600 2250
@@
 F 0 "S1" V 690 3288 50  0000 L CNN
 F 1 "A301" V 781 3288 50  0000 L CNN
-F 2 "Connector_Wire:SolderWirePad_1x02_P3.81mm_Drill1.2mm" H 750 3150 50  0001 C CNN
+F 2 "Connector_PinSocket_2.00mm:PinSocket_1x02_P2.00mm_Horizontal" H 750 3150 50  0001 C CNN
 F 3 "" H 750 3150 50  0001 C CNN
 	1    750  3150
@@
 F 0 "S2" V 690 4238 50  0000 L CNN
 F 1 "A301" V 781 4238 50  0000 L CNN
-F 2 "Connector_Wire:SolderWirePad_1x02_P3.81mm_Drill1.2mm" H 750 4100 50  0001 C CNN
+F 2 "Connector_PinSocket_2.00mm:PinSocket_1x02_P2.00mm_Horizontal" H 750 4100 50  0001 C CNN
 F 3 "" H 750 4100 50  0001 C CNN
 	1    750  4100
@@
 F 0 "S4" V 2290 3288 50  0000 L CNN
 F 1 "A301" V 2381 3288 50  0000 L CNN
-F 2 "Connector_Wire:SolderWirePad_1x02_P3.81mm_Drill1.2mm" H 2350 3150 50  0001 C CNN
+F 2 "Connector_PinSocket_2.00mm:PinSocket_1x02_P2.00mm_Horizontal" H 2350 3150 50  0001 C CNN
 F 3 "" H 2350 3150 50  0001 C CNN
 	1    2350 3150
@@
 F 0 "S5" V 2290 4238 50  0000 L CNN
 F 1 "A301" V 2381 4238 50  0000 L CNN
-F 2 "Connector_Wire:SolderWirePad_1x02_P3.81mm_Drill1.2mm" H 2350 4100 50  0001 C CNN
+F 2 "Connector_PinSocket_2.00mm:PinSocket_1x02_P2.00mm_Horizontal" H 2350 4100 50  0001 C CNN
 F 3 "" H 2350 4100 50  0001 C CNN
 	1    2350 4100
@@
 F 0 "S3" V 690 5138 50  0000 L CNN
 F 1 "A301" V 781 5138 50  0000 L CNN
-F 2 "Connector_Wire:SolderWirePad_1x02_P3.81mm_Drill1.2mm" H 750 5000 50  0001 C CNN
+F 2 "Connector_PinSocket_2.00mm:PinSocket_1x02_P2.00mm_Horizontal" H 750 5000 50  0001 C CNN
 F 3 "" H 750 5000 50  0001 C CNN
 	1    750  5000
@@
 F 0 "S6" V 2290 5138 50  0000 L CNN
 F 1 "A301" V 2381 5138 50  0000 L CNN
-F 2 "Connector_Wire:SolderWirePad_1x02_P3.81mm_Drill1.2mm" H 2350 5000 50  0001 C CNN
+F 2 "Connector_PinSocket_2.00mm:PinSocket_1x02_P2.00mm_Horizontal" H 2350 5000 50  0001 C CNN
 F 3 "" H 2350 5000 50  0001 C CNN
 	1    2350 5000
@@
 	1    0    0    -1
 $EndComp
-Text Label 800  800  2    50   ~ 0
-Source
 Text Label 5650 1050 2    50   ~ 0
 Source
@@
 	1    0    0    -1
 $EndComp
+Text Label 1650 800  1    50   ~ 0
+Source
+$Comp
+L Device:CP C10
+U 1 1 5D1AF191
+P 1450 950
+F 0 "C10" H 1568 996 50  0000 L CNN
+F 1 "470uF" H 1568 905 50  0000 L CNN
+F 2 "Capacitor_THT:CP_Radial_D5.0mm_P2.50mm" H 1488 800 50  0001 C CNN
+F 3 "" H 1450 950 50  0001 C CNN
+	1    1450 950
+	1    0    0    -1
+$EndComp
+Wire Wire Line
+	1450 1100 1450 1200
+Connection ~ 1450 1200
+Wire Wire Line
+	1450 1200 800  1200
+Connection ~ 1450 800
+Wire Wire Line
+	1450 800  1700 800
 $EndSCHEMATC
